Commit message: Exercícios 1.1 e 1.2 de sensores

File: src/model_description/model_description/urdf/robot.urdf (robot description, URDF)
Before this commit: robot meu_robo, 4 links, 3 joints
Links:
- added link camera_link; visual box size=0.06 0.06 0.04
- added link gps_link; visual cylinder length=0.015 radius=0.025
- added link imu_link; visual box size=0.04 0.04 0.02
- added link lidar_link; visual cylinder length=0.035 radius=0.07
Joints:
- added joint camera_joint: type fixed, parent base_link, child camera_link, origin xyz=0.21 0 0.14 rpy=0 0 0
- added joint gps_joint: type fixed, parent base_link, child gps_link, origin xyz=-0.10 0 0.20
- added joint imu_joint: type fixed, parent base_link, child imu_link, origin xyz=0.10 0 0.20
- added joint lidar_joint: type fixed, parent base_link, child lidar_link, origin xyz=0.12 0 0.19
